File: Schraeg/Schraeg.kicad_pcb (KiCad board)
At the start: 2 copper layers, 84.5 x 128.5 mm, 108 parts, among them U1 TL074, U2 TL074, U3 V2164, U4 TL074, U5 TL074

Commit message: v0.2.2 BOM+POS+JLC placeholder
Parts:
- removed svg2mod: G***, Schraeg:Schraeg Panel Graphics Inkscape
Other:
- board size 84.5 x 128.5 mm -> 39.5 x 110.9 mm
- board text added: "JLCJLCJLCJLC"
- board text removed: "- | +"
