File: Schraeg/Schraeg.kicad_sch (KiCad schematic)
At the start: 54 parts, among them U1 TL074, U2 TL074, U3 V2164

Commit message: v0.2.2 BOM+POS+JLC placeholder
Parts:
- C2, C4, C5, C6: LCSC (none) -> C96446
Changed lines of the file:
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@@
       (effects (font (size 1.27 1.27)) hide)
     )
-    (property "Datasheet" "~" (id 3) (at 113.03 31.75 0)
+    (property "Datasheet" "https://datasheet.lcsc.com/lcsc/1811110921_Samsung-Electro-Mechanics-CL10A106MA8NRNC_C96446.pdf" (id 3) (at 113.03 31.75 0)
       (effects (font (size 1.27 1.27)) hide)
     )
     (property "Mouser" "647-UCQ1V100MCL1GB" (id 4) (at 113.03 31.75 0)
+      (effects (font (size 1.27 1.27)) hide)
+    )
+    (property "LCSC" "C96446" (id 5) (at 113.03 31.75 0)
       (effects (font (size 1.27 1.27)) hide)
     )
@@
       (effects (font (size 1.27 1.27)) hide)
     )
-    (property "Datasheet" "~" (id 3) (at 232.41 25.4 0)
+    (property "Datasheet" "https://datasheet.lcsc.com/lcsc/1811110921_Samsung-Electro-Mechanics-CL10A106MA8NRNC_C96446.pdf" (id 3) (at 232.41 25.4 0)
       (effects (font (size 1.27 1.27)) hide)
     )
     (property "Mouser" "647-UCQ1V100MCL1GB" (id 4) (at 232.41 25.4 0)
+      (effects (font (size 1.27 1.27)) hide)
+    )
+    (property "LCSC" "C96446" (id 5) (at 232.41 25.4 0)
       (effects (font (size 1.27 1.27)) hide)
     )
@@
       (effects (font (size 1.27 1.27)) hide)
     )
-    (property "Datasheet" "~" (id 3) (at 232.41 43.18 0)
+    (property "Datasheet" "https://datasheet.lcsc.com/lcsc/1811110921_Samsung-Electro-Mechanics-CL10A106MA8NRNC_C96446.pdf" (id 3) (at 232.41 43.18 0)
       (effects (font (size 1.27 1.27)) hide)
     )
     (property "Mouser" "647-UCQ1V100MCL1GB" (id 4) (at 232.41 43.18 0)
+      (effects (font (size 1.27 1.27)) hide)
+    )
+    (property "LCSC" "C96446" (id 5) (at 232.41 43.18 0)
       (effects (font (size 1.27 1.27)) hide)
     )
@@
       (effects (font (size 1.27 1.27)) hide)
     )
-    (property "Datasheet" "~" (id 3) (at 232.41 60.96 0)
+    (property "Datasheet" "https://datasheet.lcsc.com/lcsc/1811110921_Samsung-Electro-Mechanics-CL10A106MA8NRNC_C96446.pdf" (id 3) (at 232.41 60.96 0)
       (effects (font (size 1.27 1.27)) hide)
     )
@@
       (effects (font (size 1.27 1.27)) hide)
     )
+    (property "LCSC" "C96446" (id 5) (at 232.41 60.96 0)
+      (effects (font (size 1.27 1.27)) hide)
+    )
